File: kicad/sepsepkbd.kicad_sch (KiCad schematic)
At the start: 14 parts, among them J1 Conn_01x10_Pin, J2 Conn_01x03_Pin, J3 MJ-4PP-9, J4 Conn_01x08_Pin, SW1 SW_PUSH, SW2 SW_PUSH, SW3 SW_PUSH, U1 RP2040-Zero

Commit message: additional silk on both sides
Parts:
- J1: footprint Connector_PinHeader_2.54mm:PinHeader_1x10_P2.54mm_Vertical -> sepsepkbd:PinHeader_1x10_P2.54mm_Vertical
- J2: footprint Connector_PinHeader_2.54mm:PinHeader_1x03_P2.54mm_Vertical -> sepsepkbd:PinHeader_1x03_P2.54mm_Vertical
- J4: footprint Connector_PinHeader_2.54mm:PinHeader_1x08_P2.54mm_Vertical -> sepsepkbd:PinHeader_1x08_P2.54mm_Vertical
Changed lines of the file:
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@@
 			)
 		)
-		(property "Footprint" "Connector_PinHeader_2.54mm:PinHeader_1x10_P2.54mm_Vertical"
+		(property "Footprint" "sepsepkbd:PinHeader_1x10_P2.54mm_Vertical"
 			(at 40.64 92.71 0)
 			(effects
@@
 			)
 		)
-		(property "Footprint" "Connector_PinHeader_2.54mm:PinHeader_1x08_P2.54mm_Vertical"
+		(property "Footprint" "sepsepkbd:PinHeader_1x08_P2.54mm_Vertical"
 			(at 115.57 88.9 0)
 			(effects
@@
 			)
 		)
-		(property "Footprint" "Connector_PinHeader_2.54mm:PinHeader_1x03_P2.54mm_Vertical"
+		(property "Footprint" "sepsepkbd:PinHeader_1x03_P2.54mm_Vertical"
 			(at 66.04 92.71 0)
 			(effects
